Commit message: fixed camera rotation direction

File: src/camera_description/urdf/camera.urdf (robot description, URDF)
Before this commit: robot camera, 11 links, 10 joints
Links:
- removed link camera_base
- added link urdf_camera_base
Joints:
- joint joint_9: parent camera_base -> urdf_camera_base
